File: kicad/thermostat-v3.kicad_sch (KiCad schematic)
At the start: 100 parts, among them J1 HVAC R C W Y G, J2 USB-C, J3 Stemma QT, J4 2.9in EPD FPC, Q1 AO3400A, Q2 T405-600B, Q3 T405-600B, Q4 T405-600B, SW1 RESET, SW2 BOOT, SW3 UP, SW4 DOWN, SW5 MODE, U1 LMR16006XDDCR, U2 USBLC6-2SC6, U3 ESP32-C6-WROOM-1-N8, U4 STWD100NYWY3F, U5 SHT40-AD1B, U6 MOC3063S, U7 MOC3063S, U8 MOC3063S

Commit message: Rev 13: Ferdinand review fixes - opto-gap + 0.6mm HV/LV clearance rules and reroutes, neutral footprint names, MB10S symbol pins, USB silk note, part-plan rewrite
Parts:
- C43: footprint Capacitor_THT:CP_Radial_D8.0mm_P3.50mm -> tstat:CP_Radial_D8.0mm_P3.50mm
- D1: symbol Diode_Bridge:MB2S -> tstat:BRIDGE_MB10S
- D2: footprint tstat:SMB_SMBJ40A -> tstat:D_SMB_TVS
- J2: footprint Connector_USB:USB_C_Receptacle_HRO_TYPE-C-31-M-12 -> tstat:USB_C_Receptacle_HRO_TYPE-C-31-M-12
- Q2, Q3, Q4: footprint tstat:TO-252_BT136S -> tstat:TO-252-2_TRIAC_DPAK
- TP1, TP2, TP3, TP4: footprint TestPoint:TestPoint_Pad_D1.5mm -> tstat:TestPoint_Pad_D1.5mm
Other:
- moved on the sheet: C1, C2, C3, C4, C41, C42, C43, C5, D2, D4, L1, R1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
